File: board/board.kicad_pcb (KiCad board)
At the start: 2 copper layers, 21 x 13 mm, 1 part

Commit message: initial
Parts:
- added C1: 100nF, Capacitor_SMD:C_0603_1608Metric, F.Cu at (152.2, 93.2)
- added C2: 220nF, Capacitor_SMD:C_0603_1608Metric, F.Cu at (147.5, 114.8)
- added C3: 100nF, Capacitor_SMD:C_0603_1608Metric, F.Cu at (150.5, 114.8)
- added C4: 100nF, Capacitor_SMD:C_0603_1608Metric, F.Cu at (149.0, 114.7)
- added J1: 002_SPI, on_edge:on_edge_2x05_device, F.Cu at (140.0, 96.5)
- added J2: 007_ADC, on_edge:on_edge_2x05_host, F.Cu at (161.0, 96.5)
- added J3: 007_ADC, on_edge:on_edge_2x05_host, F.Cu at (161.0, 112.5)
- added U1: ADS131M03, Package_DFN_QFN:WQFN-20-1EP_3x3mm_P0.4mm_EP1.7x1.7mm, F.Cu at (149.0, 110.0)
- added X1: 8MhZ, Oscillator:Oscillator_SMD_EuroQuartz_XO32-4Pin_3.2x2.5mm, F.Cu at (144.4, 114.4)
- moved LOGO1 19.2 mm to (169.2, 99.0)
Routing:
- net GND: track 0.00 -> 64.8 mm, vias 0 -> 7
- net /3.3V: track 0.00 -> 58.3 mm, vias 0 -> 3
- net /5V: track 0.00 -> 36.7 mm
- net /adc/MOSI: track 0.00 -> 21.9 mm
- net /adc/CS: track 0.00 -> 20.4 mm, vias 0 -> 1
- net /adc/MISO: track 0.00 -> 20.1 mm, vias 0 -> 2
- net /adc//RESET: track 0.00 -> 19.1 mm, vias 0 -> 1
- net /adc/AD3+: track 0.00 -> 18.1 mm
- net /adc/SCLK: track 0.00 -> 17.8 mm, vias 0 -> 2
- net /adc/AD3-: track 0.00 -> 16.1 mm, vias 0 -> 2
- net /adc//DRDY: track 0.00 -> 15.7 mm, vias 0 -> 2
- net /adc/AD2+: track 0.00 -> 13.5 mm, vias 0 -> 2
- net /adc/AD1-: track 0.00 -> 11.1 mm, vias 0 -> 2
- net /adc/AD2-: track 0.00 -> 9.08 mm, vias 0 -> 1
- net /adc/AD1+: track 0.00 -> 8.89 mm
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Other:
- board size 21 x 13 mm -> 21 x 29 mm
