File: board/board.kicad_sch (KiCad schematic)
At the start: 1 part

Commit message: initial
Parts:
- added J1: 002_SPI, on_edge:on_edge_2x05_device, symbol put_on_edge:002_SPI
- added J2, J3: 007_ADC, on_edge:on_edge_2x05_host, symbol put_on_edge:007_ADC
Connections:
- new net 3.3V: J1.9 (3.3V), J2.9 (3.3V), J3.9 (3.3V)
- new net 5V: J1.10 (5V), J2.10 (5V), J3.10 (5V)
- new net GND: J1.1 (GND), J2.1 (GND), J3.1 (GND)
- new net adc/AD1+: J3.3 (ADC0)
- new net adc/AD1-: J3.4 (ADC1)
- new net adc/AD2+: J3.5 (ADC2)
- new net adc/AD2-: J3.6 (ADC3)
- new net adc/AD3+: J2.3 (ADC0)
- new net adc/AD3-: J2.4 (ADC1)
- new net adc/CS: J1.6 (CS)
- new net adc/MISO: J1.3 (MISO)
- new net adc/MOSI: J1.2 (MOSI)
- new net adc/SCLK: J1.4 (SCLK)
- new net adc//DRDY: J1.5 (INT)
- new net adc//RESET: J1.8 (~{RESET})
- no-connect marks 0 -> 5
Other:
- sheet implementation renamed adc
- sheet adc: file implementation.kicad_sch -> adc.kicad_sch
- sheet adc ports: added 3.3V, AD1+, AD1-, AD2+, AD2-, AD3+, AD3-, CS, GND, MISO, MOSI, SCLK, /DRDY, /RESET; removed none
- note removed: "Input connectors go here"
- note removed: "Output connectors go here"
